File: Action_Level/PCB/Action_Card_Communication-Part.sch (KiCad schematic (older format))
At the start: 8 parts, among them U1 txb0108

Commit message: End of the schematic
Parts:
- C15, C16: renamed from C?; footprint (none) -> Capacitor_SMD:C_1206_3216Metric_Pad1.42x1.75mm_HandSolder
- J1, J2: renamed from J?; footprint (none) -> Connector_Molex:Molex_KK-254_1x03_P2.54mm_Horizontal
- J3: renamed from J?; footprint (none) -> Connector_Molex:Molex_KK-254_1x04_P2.54mm_Horizontal
- Rp1, Rp2: footprint (none) -> Resistor_SMD:R_1206_3216Metric_Pad1.42x1.75mm_HandSolder
- U1: footprint (none) -> Package_SO:TSSOP-20_4.4x6.5mm_P0.65mm
Changed lines of the file:
@@
 $EndDescr
 $Comp
-L Connector_Generic:Conn_01x03 J?
+L Connector_Generic:Conn_01x03 J2
 U 1 1 5C798AB0
 P 4175 3350
-F 0 "J?" H 4250 3300 50  0000 L CNN
+F 0 "J2" H 4250 3300 50  0000 L CNN
 F 1 "Conn_01x03" H 4250 3425 50  0000 L CNN
-F 2 "" H 4175 3350 50  0001 C CNN
+F 2 "Connector_Molex:Molex_KK-254_1x03_P2.54mm_Horizontal" H 4175 3350 50  0001 C CNN
 F 3 "~" H 4175 3350 50  0001 C CNN
 	1    4175 3350
@@
 $EndComp
 $Comp
-L Connector_Generic:Conn_01x03 J?
+L Connector_Generic:Conn_01x03 J1
 U 1 1 5C798BD1
 P 2900 3350
-F 0 "J?" H 3025 3325 50  0000 C CNN
+F 0 "J1" H 3025 3325 50  0000 C CNN
 F 1 "Conn_01x03" H 3225 3425 50  0000 C CNN
-F 2 "" H 2900 3350 50  0001 C CNN
+F 2 "Connector_Molex:Molex_KK-254_1x03_P2.54mm_Horizontal" H 2900 3350 50  0001 C CNN
 F 3 "~" H 2900 3350 50  0001 C CNN
 	1    2900 3350
@@
 $EndComp
 $Comp
-L power:GND #PWR?
+L power:GND #PWR0159
 U 1 1 5C798D76
 P 3100 3450
-F 0 "#PWR?" H 3100 3200 50  0001 C CNN
+F 0 "#PWR0159" H 3100 3200 50  0001 C CNN
 F 1 "GND" H 3105 3277 50  0000 C CNN
 F 2 "" H 3100 3450 50  0001 C CNN
@@
 $EndComp
 $Comp
-L power:GND #PWR?
+L power:GND #PWR0160
 U 1 1 5C798D8C
 P 3975 3450
-F 0 "#PWR?" H 3975 3200 50  0001 C CNN
+F 0 "#PWR0160" H 3975 3200 50  0001 C CNN
 F 1 "GND" H 3980 3277 50  0000 C CNN
 F 2 "" H 3975 3450 50  0001 C CNN
@@
 SCL(5V)
 $Comp
-L power:+5V #PWR?
+L power:+5V #PWR0161
 U 1 1 5C799057
 P 3275 2375
-F 0 "#PWR?" H 3275 2225 50  0001 C CNN
+F 0 "#PWR0161" H 3275 2225 50  0001 C CNN
 F 1 "+5V" H 3290 2548 50  0000 C CNN
 F 2 "" H 3275 2375 50  0001 C CNN
@@
 $EndComp
 $Comp
-L power:+5V #PWR?
+L power:+5V #PWR0162
 U 1 1 5C799095
 P 3875 2375
-F 0 "#PWR?" H 3875 2225 50  0001 C CNN
+F 0 "#PWR0162" H 3875 2225 50  0001 C CNN
 F 1 "+5V" H 3890 2548 50  0000 C CNN
 F 2 "" H 3875 2375 50  0001 C CNN
@@
 F 0 "Rp1" H 3075 2575 50  0000 L CNN
 F 1 "10k" V 3275 2450 50  0000 L CNN
-F 2 "" V 3205 2525 50  0001 C CNN
+F 2 "Resistor_SMD:R_1206_3216Metric_Pad1.42x1.75mm_HandSolder" V 3205 2525 50  0001 C CNN
 F 3 "~" H 3275 2525 50  0001 C CNN
 	1    3275 2525
@@
 F 0 "Rp2" H 3675 2575 50  0000 L CNN
 F 1 "10k" V 3875 2450 50  0000 L CNN
-F 2 "" V 3805 2525 50  0001 C CNN
+F 2 "Resistor_SMD:R_1206_3216Metric_Pad1.42x1.75mm_HandSolder" V 3805 2525 50  0001 C CNN
 F 3 "~" H 3875 2525 50  0001 C CNN
 	1    3875 2525
@@
 F 0 "U1" H 3025 3125 50  0000 C CNN
 F 1 "txb0108" H 3025 3034 50  0000 C CNN
-F 2 "" H 2675 2850 50  0001 C CNN
+F 2 "Package_SO:TSSOP-20_4.4x6.5mm_P0.65mm" H 2675 2850 50  0001 C CNN
 F 3 "http://www.ti.com/lit/ds/symlink/txb0108.pdf" H 2675 2850 50  0001 C CNN
 	1    3025 2900
@@
 F 0 "U1" H 4125 2685 50  0000 C CNN
 F 1 "txb0108" H 4125 2776 50  0000 C CNN
-F 2 "" H 3775 2850 50  0001 C CNN
+F 2 "Package_SO:TSSOP-20_4.4x6.5mm_P0.65mm" H 3775 2850 50  0001 C CNN
 F 3 "http://www.ti.com/lit/ds/symlink/txb0108.pdf" H 3775 2850 50  0001 C CNN
 	2    4125 2900
@@
 F 0 "U1" H 3525 4225 50  0000 C CNN
 F 1 "txb0108" H 3525 4134 50  0000 C CNN
-F 2 "" H 3175 3950 50  0001 C CNN
+F 2 "Package_SO:TSSOP-20_4.4x6.5mm_P0.65mm" H 3175 3950 50  0001 C CNN
 F 3 "http://www.ti.com/lit/ds/symlink/txb0108.pdf" H 3175 3950 50  0001 C CNN
 	9    3525 4000
@@
 $EndComp
 $Comp
-L power:+5V #PWR?
+L power:+5V #PWR0163
 U 1 1 5C799857
 P 4075 4000
-F 0 "#PWR?" H 4075 3850 50  0001 C CNN
+F 0 "#PWR0163" H 4075 3850 50  0001 C CNN
 F 1 "+5V" H 4090 4173 50  0000 C CNN
 F 2 "" H 4075 4000 50  0001 C CNN
@@
 $EndComp
 $Comp
-L power:GND #PWR?
+L power:GND #PWR0164
 U 1 1 5C79987E
 P 4075 4300
-F 0 "#PWR?" H 4075 4050 50  0001 C CNN
+F 0 "#PWR0164" H 4075 4050 50  0001 C CNN
 F 1 "GND" H 4080 4127 50  0000 C CNN
 F 2 "" H 4075 4300 50  0001 C CNN
@@
 $EndComp
 $Comp
-L power:+3V3 #PWR?
+L power:+3V3 #PWR0165
 U 1 1 5C7998C6
 P 2975 4000
-F 0 "#PWR?" H 2975 3850 50  0001 C CNN
+F 0 "#PWR0165" H 2975 3850 50  0001 C CNN
 F 1 "+3V3" H 2990 4173 50  0000 C CNN
 F 2 "" H 2975 4000 50  0001 C CNN
@@
 $EndComp
 $Comp
-L Device:C C?
+L Device:C C15
 U 1 1 5C79996F
 P 2975 4150
-F 0 "C?" H 2750 4200 50  0000 L CNN
+F 0 "C15" H 2750 4200 50  0000 L CNN
 F 1 "0.1u" H 2700 4125 50  0000 L CNN
-F 2 "" H 3013 4000 50  0001 C CNN
+F 2 "Capacitor_SMD:C_1206_3216Metric_Pad1.42x1.75mm_HandSolder" H 3013 4000 50  0001 C CNN
 F 3 "~" H 2975 4150 50  0001 C CNN
 	1    2975 4150
@@
 $EndComp
 $Comp
-L Device:C C?
+L Device:C C16
 U 1 1 5C799A96
 P 4075 4150
-F 0 "C?" H 4200 4200 50  0000 L CNN
+F 0 "C16" H 4200 4200 50  0000 L CNN
 F 1 "0.1u" H 4200 4125 50  0000 L CNN
-F 2 "" H 4113 4000 50  0001 C CNN
+F 2 "Capacitor_SMD:C_1206_3216Metric_Pad1.42x1.75mm_HandSolder" H 4113 4000 50  0001 C CNN
 F 3 "~" H 4075 4150 50  0001 C CNN
 	1    4075 4150
@@
 Connection ~ 4075 4000
 $Comp
-L power:GND #PWR?
+L power:GND #PWR0166
 U 1 1 5C799C12
 P 3875 4100
-F 0 "#PWR?" H 3875 3850 50  0001 C CNN
+F 0 "#PWR0166" H 3875 3850 50  0001 C CNN
 F 1 "GND" H 3880 3927 50  0000 C CNN
 F 2 "" H 3875 4100 50  0001 C CNN
@@
 	3100 4000 2975 4000
 $Comp
-L power:GND #PWR?
+L power:GND #PWR0167
 U 1 1 5C799CFE
 P 2975 4300
-F 0 "#PWR?" H 2975 4050 50  0001 C CNN
+F 0 "#PWR0167" H 2975 4050 50  0001 C CNN
 F 1 "GND" H 2980 4127 50  0000 C CNN
 F 2 "" H 2975 4300 50  0001 C CNN
@@
 SCL(3V3)
 $Comp
-L Connector_Generic:Conn_01x04 J?
+L Connector_Generic:Conn_01x04 J3
 U 1 1 5C79B355
 P 7625 3400
-F 0 "J?" H 7545 2975 50  0000 C CNN
+F 0 "J3" H 7545 2975 50  0000 C CNN
 F 1 "Conn_01x04" H 7545 3066 50  0000 C CNN
-F 2 "" H 7625 3400 50  0001 C CNN
+F 2 "Connector_Molex:Molex_KK-254_1x04_P2.54mm_Horizontal" H 7625 3400 50  0001 C CNN
 F 3 "~" H 7625 3400 50  0001 C CNN
 	1    7625 3400
@@
 	7825 3400 8475 3400
 $Comp
-L power:GND #PWR?
+L power:GND #PWR0168
 U 1 1 5C79B83A
 P 7825 3500
-F 0 "#PWR?" H 7825 3250 50  0001 C CNN
+F 0 "#PWR0168" H 7825 3250 50  0001 C CNN
 F 1 "GND" H 7830 3327 50  0000 C CNN
 F 2 "" H 7825 3500 50  0001 C CNN
