File: Action_Level/PCB/Action_Card_uC.sch (KiCad schematic (older format))
At the start: 9 parts

Commit message: End of the schematic
Parts:
- added C5, C6: 0.1u, Capacitor_SMD:C_1206_3216Metric_Pad1.42x1.75mm_HandSolder, symbol Device:C
- added U2: txb0108, Package_SO:TSSOP-20_4.4x6.5mm_P0.65mm, symbol stm32f042k6tx:txb0108
- C1, C2, C3, C4: renamed from C?; footprint (none) -> Capacitor_SMD:C_1206_3216Metric_Pad1.42x1.75mm_HandSolder
- D9: renamed from D?; footprint (none) -> LED_SMD:LED_1206_3216Metric_Pad1.42x1.75mm_HandSolder
- R1, R2: renamed from R?; footprint (none) -> Resistor_SMD:R_1206_3216Metric_Pad1.42x1.75mm_HandSolder
- SW1: renamed from SW?; footprint (none) -> Connector_PinHeader_2.54mm:PinHeader_1x03_P2.54mm_Vertical; symbol Switch:SW_DPDT_x2 -> Device:Jumper_NC_Dual
- U3: renamed from U?; footprint (none) -> Package_QFP:LQFP-32_7x7mm_P0.8mm
Connections:
- net labels added: +5V, DIR_PaP, EN_DC_EXT(3V3), EN_DC_INT(3V3), FC_LB, FC_LT, FC_RB, FC_RT, PWM_L-DC_EXT(3V3), PWM_L-DC_INT(3V3), PWM_R-DC_EXT(3V3), PWM_R-DC_INT(3V3), SENSOR_AR, SENSOR_AV, STEP_PaP, ~EN~_PaP-L, ~EN~_PaP-R
- net labels removed: DIR-PaP, EN-PaP, STEP-PaP
- wire segments 19 -> 66
- no-connect marks 2 -> 4
Other:
- note added: "(Sorties en 3V3)"
- note added: "Conversion des commandes 3V3 -> 5V\n"
- note added: "Position GND pour Flasher"
