File: Action_Level/PCB/Action_Card.sch (KiCad schematic (older format))
At the start: 0 parts

Commit message: End of the schematic
Connections:
- wire segments 11 -> 29
Changed lines of the file:
@@
 F5 "SDA(3V3)" I L 4700 4150 50
 F6 "SCL(3V3)" I L 4700 4225 50
+F7 "PWM_L-DC_INT" O R 6475 2675 50
+F8 "PWM_R-DC_INT" O R 6475 2750 50
+F9 "EN_DC_INT" O R 6475 2600 50
+F10 "PWM_L-DC_EXT" O R 6475 3225 50
+F11 "PWM_R-DC_EXT" O R 6475 3300 50
+F12 "EN_DC_EXT" O R 6475 3150 50
+F13 "STEP_PaP" O R 6475 4525 50
+F14 "DIR_PaP" O R 6475 4600 50
+F15 "~EN~_PaP-R" O R 6475 4250 50
+F16 "~EN~_PaP-L" O R 6475 4350 50
+F17 "FC_LT" I L 4700 2925 50
+F18 "FC_RT" I L 4700 3000 50
+F19 "FC_LB" I L 4700 3075 50
+F20 "FC_RB" I L 4700 3150 50
+F21 "SENSOR_AV" I L 4700 3350 50
+F22 "SENSOR_AR" I L 4700 3425 50
 $EndSheet
 $Sheet
@@
 F0 "DC-Motor-Part" 50
 F1 "Action_Card_DC-Motor-Part.sch" 50
-F2 "EN_DC_INT" I L 7575 2575 50
+F2 "EN_DC_INT" I L 7575 2600 50
+F3 "PWM_L-DC_INT" I L 7575 2675 50
+F4 "PWM_R-DC_INT" I L 7575 2750 50
+F5 "EN_DC_EXT" I L 7575 3150 50
+F6 "PWM_L-DC_EXT" I L 7575 3225 50
+F7 "PWM_R-DC_EXT" I L 7575 3300 50
 $EndSheet
 $Sheet
@@
 F0 "Stepper-Motor-Part" 50
 F1 "Action_Card_Stepper-Motor-Part.sch" 50
+F2 "DIR_PaP" I L 7575 4775 50
+F3 "STEP_PaP" I L 7575 4700 50
+F4 "~EN~_PaP-R" I L 7575 4375 50
+F5 "~EN~_PaP-L" I L 7575 4475 50
 $EndSheet
 Wire Wire Line
@@
 F0 "Sensors-Part" 50
 F1 "Action_Card_Sensors-Part.sch" 50
+F2 "FC_LT" O R 4050 2925 50
+F3 "FC_RT" O R 4050 3000 50
+F4 "FC_LB" O R 4050 3075 50
+F5 "FC_RB" O R 4050 3150 50
+F6 "SENSOR_AV" O R 4050 3350 50
+F7 "SENSOR_AR" O R 4050 3425 50
 $EndSheet
+Wire Wire Line
+	7575 4375 7175 4375
+Wire Wire Line
+	7175 4375 7175 4250
+Wire Wire Line
+	7175 4250 6475 4250
+Wire Wire Line
+	6475 4350 7075 4350
+Wire Wire Line
+	7075 4350 7075 4475
+Wire Wire Line
+	7075 4475 7575 4475
+Wire Wire Line
+	6475 4525 7000 4525
+Wire Wire Line
+	7000 4525 7000 4700
+Wire Wire Line
+	7000 4700 7575 4700
+Wire Wire Line
+	7575 4775 6925 4775
+Wire Wire Line
+	6925 4775 6925 4600
+Wire Wire Line
+	6925 4600 6475 4600
+Wire Wire Line
+	4050 2925 4700 2925
+Wire Wire Line
+	4700 3000 4050 3000
+Wire Wire Line
+	4050 3075 4700 3075
+Wire Wire Line
+	4700 3150 4050 3150
+Wire Wire Line
+	4050 3350 4700 3350
+Wire Wire Line
+	4050 3425 4700 3425
 $EndSCHEMATC

Commit message: First big step in route
Parts:
- added U10, U11, U12, U13: Trou-3, maxon:Trou-3, symbol Propulsion_control:Trou-3
Connections:
- net labels added: GND
- wire segments 29 -> 37
Changed lines of the file:
@@
 Wire Wire Line
 	4050 3425 4700 3425
+$Comp
+L Propulsion_control:Trou-3 U10
+U 1 1 5C8EDF38
+P 1750 5825
+F 0 "U10" H 1878 5878 60  0000 L CNN
+F 1 "Trou-3" H 1878 5772 60  0000 L CNN
+F 2 "maxon:Trou-3" H 1750 5825 60  0001 C CNN
+F 3 "" H 1750 5825 60  0000 C CNN
+	1    1750 5825
+	1    0    0    -1
+$EndComp
+$Comp
+L Propulsion_control:Trou-3 U11
+U 1 1 5C8EDF90
+P 1750 6050
+F 0 "U11" H 1878 6103 60  0000 L CNN
+F 1 "Trou-3" H 1878 5997 60  0000 L CNN
+F 2 "maxon:Trou-3" H 1750 6050 60  0001 C CNN
+F 3 "" H 1750 6050 60  0000 C CNN
+	1    1750 6050
+	1    0    0    -1
+$EndComp
+$Comp
+L Propulsion_control:Trou-3 U12
+U 1 1 5C8EDFBA
+P 1750 6275
+F 0 "U12" H 1878 6328 60  0000 L CNN
+F 1 "Trou-3" H 1878 6222 60  0000 L CNN
+F 2 "maxon:Trou-3" H 1750 6275 60  0001 C CNN
+F 3 "" H 1750 6275 60  0000 C CNN
+	1    1750 6275
+	1    0    0    -1
+$EndComp
+$Comp
+L Propulsion_control:Trou-3 U13
+U 1 1 5C8EDFD7
+P 1750 6500
+F 0 "U13" H 1878 6553 60  0000 L CNN
+F 1 "Trou-3" H 1878 6447 60  0000 L CNN
+F 2 "maxon:Trou-3" H 1750 6500 60  0001 C CNN
+F 3 "" H 1750 6500 60  0000 C CNN
+	1    1750 6500
+	1    0    0    -1
+$EndComp
+$Comp
+L power:GND #PWR01
+U 1 1 5C8EE033
+P 1300 6650
+F 0 "#PWR01" H 1300 6400 50  0001 C CNN
+F 1 "GND" H 1305 6477 50  0000 C CNN
+F 2 "" H 1300 6650 50  0001 C CNN
+F 3 "" H 1300 6650 50  0001 C CNN
+	1    1300 6650
+	1    0    0    -1
+$EndComp
+Wire Wire Line
+	1450 5825 1300 5825
+Wire Wire Line
+	1300 5825 1300 6050
+Wire Wire Line
+	1450 6050 1300 6050
+Connection ~ 1300 6050
+Wire Wire Line
+	1300 6050 1300 6275
+Wire Wire Line
+	1450 6275 1300 6275
+Connection ~ 1300 6275
+Wire Wire Line
+	1300 6275 1300 6500
+Wire Wire Line
+	1450 6500 1300 6500
+Connection ~ 1300 6500
+Wire Wire Line
+	1300 6500 1300 6650
 $EndSCHEMATC
