File: Action_Level/PCB/Action_Card_DC-Motor-Part.sch (KiCad schematic (older format))
At the start: 15 parts

Commit message: End of the schematic
Parts:
- C13: renamed from C?; footprint (none) -> Capacitor_SMD:C_1206_3216Metric_Pad1.42x1.75mm_HandSolder
- C14: renamed from C?; footprint (none) -> Capacitor_THT:CP_Radial_D8.0mm_P3.50mm
- D1, D2, D3, D4, D5, D6, D7, D8: renamed from D?; footprint (none) -> Diode_THT:D_DO-35_SOD27_P10.16mm_Horizontal
- J_DC_EXT1: renamed from J_DC_EXT; footprint (none) -> Connector_Molex:Molex_KK-254_1x02_P2.54mm_Horizontal
- J_DC_INT1: renamed from J_DC_INT; footprint (none) -> Connector_Molex:Molex_KK-254_1x02_P2.54mm_Horizontal
- R12, R13: renamed from R?; footprint (none) -> Resistor_SMD:R_1206_3216Metric_Pad1.42x1.75mm_HandSolder
- gave numbers to parts that had none: 1
Changed lines of the file:
@@
 $EndDescr
 $Comp
-L power:+5VA #PWR?
+L power:+5VA #PWR0144
 U 1 1 5C7A472D
 P 5800 1975
-F 0 "#PWR?" H 5800 1825 50  0001 C CNN
+F 0 "#PWR0144" H 5800 1825 50  0001 C CNN
 F 1 "+5VA" H 5815 2148 50  0000 C CNN
 F 2 "" H 5800 1975 50  0001 C CNN
@@
 $EndComp
 $Comp
-L power:+5V #PWR?
+L power:+5V #PWR0145
 U 1 1 5C7A4773
 P 5600 1975
-F 0 "#PWR?" H 5600 1825 50  0001 C CNN
+F 0 "#PWR0145" H 5600 1825 50  0001 C CNN
 F 1 "+5V" H 5615 2148 50  0000 C CNN
 F 2 "" H 5600 1975 50  0001 C CNN
@@
 $EndComp
 $Comp
-L power:GND #PWR?
+L power:GND #PWR0146
 U 1 1 5C7A484B
 P 5700 4150
-F 0 "#PWR?" H 5700 3900 50  0001 C CNN
+F 0 "#PWR0146" H 5700 3900 50  0001 C CNN
 F 1 "GND" H 5705 3977 50  0000 C CNN
 F 2 "" H 5700 4150 50  0001 C CNN
@@
 PWM_R-DC_INT
 $Comp
-L Connector_Generic:Conn_01x02 J_DC_INT
+L Connector_Generic:Conn_01x02 J_DC_INT1
 U 1 1 5C7A4C0F
 P 7750 2625
-F 0 "J_DC_INT" H 7830 2617 50  0000 L CNN
+F 0 "J_DC_INT1" H 7830 2617 50  0000 L CNN
 F 1 "Conn_MDC" H 7830 2526 50  0000 L CNN
-F 2 "" H 7750 2625 50  0001 C CNN
+F 2 "Connector_Molex:Molex_KK-254_1x02_P2.54mm_Horizontal" H 7750 2625 50  0001 C CNN
 F 3 "~" H 7750 2625 50  0001 C CNN
 	1    7750 2625
@@
 $EndComp
 $Comp
-L Device:D_ALT D?
+L Device:D_ALT D2
 U 1 1 5C7A4CC5
 P 7150 2425
-F 0 "D?" H 7150 2325 50  0000 C CNN
+F 0 "D2" H 7150 2325 50  0000 C CNN
 F 1 "D_ALT" H 7150 2550 50  0000 C CNN
-F 2 "" H 7150 2425 50  0001 C CNN
+F 2 "Diode_THT:D_DO-35_SOD27_P10.16mm_Horizontal" H 7150 2425 50  0001 C CNN
 F 3 "~" H 7150 2425 50  0001 C CNN
 	1    7150 2425
@@
 $EndComp
 $Comp
-L Device:D_ALT D?
+L Device:D_ALT D1
 U 1 1 5C7A4CFF
 P 6700 2425
-F 0 "D?" H 6700 2325 50  0000 C CNN
+F 0 "D1" H 6700 2325 50  0000 C CNN
 F 1 "D_ALT" H 6725 2525 50  0000 C CNN
-F 2 "" H 6700 2425 50  0001 C CNN
+F 2 "Diode_THT:D_DO-35_SOD27_P10.16mm_Horizontal" H 6700 2425 50  0001 C CNN
 F 3 "~" H 6700 2425 50  0001 C CNN
 	1    6700 2425
@@
 $EndComp
 $Comp
-L Device:D_ALT D?
+L Device:D_ALT D3
 U 1 1 5C7A4D1C
 P 6700 2900
-F 0 "D?" H 6700 3000 50  0000 C CNN
+F 0 "D3" H 6700 3000 50  0000 C CNN
 F 1 "D_ALT" H 6700 2775 50  0000 C CNN
-F 2 "" H 6700 2900 50  0001 C CNN
+F 2 "Diode_THT:D_DO-35_SOD27_P10.16mm_Horizontal" H 6700 2900 50  0001 C CNN
 F 3 "~" H 6700 2900 50  0001 C CNN
 	1    6700 2900
@@
 $EndComp
 $Comp
-L Device:D_ALT D?
+L Device:D_ALT D4
 U 1 1 5C7A4D3D
 P 7150 2900
-F 0 "D?" H 7150 3000 50  0000 C CNN
+F 0 "D4" H 7150 3000 50  0000 C CNN
 F 1 "D_ALT" H 7150 2775 50  0000 C CNN
-F 2 "" H 7150 2900 50  0001 C CNN
+F 2 "Diode_THT:D_DO-35_SOD27_P10.16mm_Horizontal" H 7150 2900 50  0001 C CNN
 F 3 "~" H 7150 2900 50  0001 C CNN
 	1    7150 2900
@@
 	7550 2725 6925 2725
 $Comp
-L power:GND #PWR?
+L power:GND #PWR0147
 U 1 1 5C7A550B
 P 7300 2425
-F 0 "#PWR?" H 7300 2175 50  0001 C CNN
+F 0 "#PWR0147" H 7300 2175 50  0001 C CNN
 F 1 "GND" H 7450 2375 50  0000 C CNN
 F 2 "" H 7300 2425 50  0001 C CNN
@@
 $EndComp
 $Comp
-L power:+5VA #PWR?
+L power:+5VA #PWR0148
 U 1 1 5C7A5522
 P 6550 2425
-F 0 "#PWR?" H 6550 2275 50  0001 C CNN
+F 0 "#PWR0148" H 6550 2275 50  0001 C CNN
 F 1 "+5VA" H 6425 2550 50  0000 C CNN
 F 2 "" H 6550 2425 50  0001 C CNN
@@
 	6925 2625 7550 2625
 $Comp
-L power:GND #PWR?
+L power:GND #PWR0149
 U 1 1 5C7A5D13
 P 7300 2900
-F 0 "#PWR?" H 7300 2650 50  0001 C CNN
+F 0 "#PWR0149" H 7300 2650 50  0001 C CNN
 F 1 "GND" H 7450 2850 50  0000 C CNN
 F 2 "" H 7300 2900 50  0001 C CNN
@@
 $EndComp
 $Comp
-L power:+5VA #PWR?
+L power:+5VA #PWR0150
 U 1 1 5C7A5E45
 P 6550 2900
-F 0 "#PWR?" H 6550 2750 50  0001 C CNN
+F 0 "#PWR0150" H 6550 2750 50  0001 C CNN
 F 1 "+5VA" H 6425 2925 50  0000 C CNN
 F 2 "" H 6550 2900 50  0001 C CNN
@@
 	6925 2725 6300 2725
 $Comp
-L Device:C C?
+L Device:C C13
 U 1 1 5C7A70A8
 P 5450 2125
-F 0 "C?" V 5300 2125 50  0000 C CNN
+F 0 "C13" V 5300 2125 50  0000 C CNN
 F 1 "0.1u" V 5375 1975 50  0000 C CNN
-F 2 "" H 5488 1975 50  0001 C CNN
+F 2 "Capacitor_SMD:C_1206_3216Metric_Pad1.42x1.75mm_HandSolder" H 5488 1975 50  0001 C CNN
 F 3 "~" H 5450 2125 50  0001 C CNN
 	1    5450 2125
@@
 $EndComp
 $Comp
-L power:GND #PWR?
+L power:GND #PWR0151
 U 1 1 5C7A719F
 P 5300 2125
-F 0 "#PWR?" H 5300 1875 50  0001 C CNN
+F 0 "#PWR0151" H 5300 1875 50  0001 C CNN
 F 1 "GND" H 5200 2000 50  0000 C CNN
 F 2 "" H 5300 2125 50  0001 C CNN
@@
 Connection ~ 5600 2125
 $Comp
-L Device:C C?
+L Device:C C14
 U 1 1 5C7A7617
 P 5950 2125
-F 0 "C?" V 6100 2125 50  0000 C CNN
+F 0 "C14" V 6100 2125 50  0000 C CNN
 F 1 "1u" V 6025 1975 50  0000 C CNN
-F 2 "" H 5988 1975 50  0001 C CNN
+F 2 "Capacitor_THT:CP_Radial_D8.0mm_P3.50mm" H 5988 1975 50  0001 C CNN
 F 3 "~" H 5950 2125 50  0001 C CNN
 	1    5950 2125
@@
 $EndComp
 $Comp
-L power:GND #PWR?
+L power:GND #PWR0152
 U 1 1 5C7A76DE
 P 6100 2125
-F 0 "#PWR?" H 6100 1875 50  0001 C CNN
+F 0 "#PWR0152" H 6100 1875 50  0001 C CNN
 F 1 "GND" H 6225 2025 50  0000 C CNN
 F 2 "" H 6100 2125 50  0001 C CNN
@@
 Connection ~ 5800 2125
 $Comp
-L Device:R R?
+L Device:R R12
 U 1 1 5C7AA441
 P 4025 2775
-F 0 "R?" H 4095 2821 50  0000 L CNN
+F 0 "R12" H 4095 2821 50  0000 L CNN
 F 1 "10k" V 4025 2700 50  0000 L CNN
-F 2 "" V 3955 2775 50  0001 C CNN
+F 2 "Resistor_SMD:R_1206_3216Metric_Pad1.42x1.75mm_HandSolder" V 3955 2775 50  0001 C CNN
 F 3 "~" H 4025 2775 50  0001 C CNN
 	1    4025 2775
@@
 $EndComp
 $Comp
-L power:GND #PWR?
+L power:GND #PWR0153
 U 1 1 5C7AA4E0
 P 4025 2925
-F 0 "#PWR?" H 4025 2675 50  0001 C CNN
+F 0 "#PWR0153" H 4025 2675 50  0001 C CNN
 F 1 "GND" H 4030 2752 50  0000 C CNN
 F 2 "" H 4025 2925 50  0001 C CNN
@@
 Moteur tapis roulant
 $Comp
-L Connector_Generic:Conn_01x02 J_DC_EXT
+L Connector_Generic:Conn_01x02 J_DC_EXT1
 U 1 1 5C8B33A7
 P 7750 3650
-F 0 "J_DC_EXT" H 7830 3642 50  0000 L CNN
+F 0 "J_DC_EXT1" H 7830 3642 50  0000 L CNN
 F 1 "Conn_MDC" H 7830 3551 50  0000 L CNN
-F 2 "" H 7750 3650 50  0001 C CNN
+F 2 "Connector_Molex:Molex_KK-254_1x02_P2.54mm_Horizontal" H 7750 3650 50  0001 C CNN
 F 3 "~" H 7750 3650 50  0001 C CNN
 	1    7750 3650
@@
 $EndComp
 $Comp
-L Device:D_ALT D?
+L Device:D_ALT D6
 U 1 1 5C8B34B6
 P 7150 3450
-F 0 "D?" H 7150 3350 50  0000 C CNN
+F 0 "D6" H 7150 3350 50  0000 C CNN
 F 1 "D_ALT" H 7150 3575 50  0000 C CNN
-F 2 "" H 7150 3450 50  0001 C CNN
+F 2 "Diode_THT:D_DO-35_SOD27_P10.16mm_Horizontal" H 7150 3450 50  0001 C CNN
 F 3 "~" H 7150 3450 50  0001 C CNN
 	1    7150 3450
@@
 $EndComp
 $Comp
-L Device:D_ALT D?
+L Device:D_ALT D5
 U 1 1 5C8B34BD
 P 6700 3450
-F 0 "D?" H 6700 3350 50  0000 C CNN
+F 0 "D5" H 6700 3350 50  0000 C CNN
 F 1 "D_ALT" H 6725 3550 50  0000 C CNN
-F 2 "" H 6700 3450 50  0001 C CNN
+F 2 "Diode_THT:D_DO-35_SOD27_P10.16mm_Horizontal" H 6700 3450 50  0001 C CNN
 F 3 "~" H 6700 3450 50  0001 C CNN
 	1    6700 3450
@@
 $EndComp
 $Comp
-L Device:D_ALT D?
+L Device:D_ALT D7
 U 1 1 5C8B34C4
 P 6700 3925
-F 0 "D?" H 6700 4025 50  0000 C CNN
+F 0 "D7" H 6700 4025 50  0000 C CNN
 F 1 "D_ALT" H 6700 3800 50  0000 C CNN
-F 2 "" H 6700 3925 50  0001 C CNN
+F 2 "Diode_THT:D_DO-35_SOD27_P10.16mm_Horizontal" H 6700 3925 50  0001 C CNN
 F 3 "~" H 6700 3925 50  0001 C CNN
 	1    6700 3925
@@
 $EndComp
 $Comp
-L Device:D_ALT D?
+L Device:D_ALT D8
 U 1 1 5C8B34CB
 P 7150 3925
-F 0 "D?" H 7150 4025 50  0000 C CNN
+F 0 "D8" H 7150 4025 50  0000 C CNN
 F 1 "D_ALT" H 7150 3800 50  0000 C CNN
-F 2 "" H 7150 3925 50  0001 C CNN
+F 2 "Diode_THT:D_DO-35_SOD27_P10.16mm_Horizontal" H 7150 3925 50  0001 C CNN
 F 3 "~" H 7150 3925 50  0001 C CNN
 	1    7150 3925
@@
 	7550 3750 6925 3750
 $Comp
-L power:GND #PWR?
+L power:GND #PWR0154
 U 1 1 5C8B34D4
 P 7300 3450
-F 0 "#PWR?" H 7300 3200 50  0001 C CNN
+F 0 "#PWR0154" H 7300 3200 50  0001 C CNN
 F 1 "GND" H 7450 3400 50  0000 C CNN
 F 2 "" H 7300 3450 50  0001 C CNN
@@
 $EndComp
 $Comp
-L power:+5VA #PWR?
+L power:+5VA #PWR0155
 U 1 1 5C8B34DA
 P 6550 3450
-F 0 "#PWR?" H 6550 3300 50  0001 C CNN
+F 0 "#PWR0155" H 6550 3300 50  0001 C CNN
 F 1 "+5VA" H 6425 3575 50  0000 C CNN
 F 2 "" H 6550 3450 50  0001 C CNN
@@
 	6925 3650 7550 3650
 $Comp
-L power:GND #PWR?
+L power:GND #PWR0156
 U 1 1 5C8B34E6
 P 7300 3925
-F 0 "#PWR?" H 7300 3675 50  0001 C CNN
+F 0 "#PWR0156" H 7300 3675 50  0001 C CNN
 F 1 "GND" H 7450 3875 50  0000 C CNN
 F 2 "" H 7300 3925 50  0001 C CNN
@@
 $EndComp
 $Comp
-L power:+5VA #PWR?
+L power:+5VA #PWR0157
 U 1 1 5C8B34EC
 P 6550 3925
-F 0 "#PWR?" H 6550 3775 50  0001 C CNN
+F 0 "#PWR0157" H 6550 3775 50  0001 C CNN
 F 1 "+5VA" H 6425 3950 50  0000 C CNN
 F 2 "" H 6550 3925 50  0001 C CNN
@@
 	4250 3625 3825 3625
 $Comp
-L Device:R R?
+L Device:R R13
 U 1 1 5C8B72FA
 P 4025 4175
-F 0 "R?" H 4095 4221 50  0000 L CNN
+F 0 "R13" H 4095 4221 50  0000 L CNN
 F 1 "10k" V 4025 4100 50  0000 L CNN
-F 2 "" V 3955 4175 50  0001 C CNN
+F 2 "Resistor_SMD:R_1206_3216Metric_Pad1.42x1.75mm_HandSolder" V 3955 4175 50  0001 C CNN
 F 3 "~" H 4025 4175 50  0001 C CNN
 	1    4025 4175
@@
 $EndComp
 $Comp
-L power:GND #PWR?
+L power:GND #PWR0158
 U 1 1 5C8B7301
 P 4025 4325
-F 0 "#PWR?" H 4025 4075 50  0001 C CNN
+F 0 "#PWR0158" H 4025 4075 50  0001 C CNN
 F 1 "GND" H 4030 4152 50  0000 C CNN
 F 2 "" H 4025 4325 50  0001 C CNN
@@
 Connection ~ 5800 4025
 $Comp
-L Driver_Motor:L293 U?
+L Driver_Motor:L293 U4
 U 1 1 5C7A467A
 P 5700 3225
-F 0 "U?" H 5400 4050 50  0000 C CNN
+F 0 "U4" H 5400 4050 50  0000 C CNN
 F 1 "L293" H 5950 2850 50  0000 C CNN
 F 2 "Package_DIP:DIP-16_W7.62mm" H 5950 2475 50  0001 L CNN

Commit message: First big step in route
Parts:
- removed D1, D2, D3, D4, D5, D6, D7, D8: D_ALT, Diode_THT:D_DO-35_SOD27_P10.16mm_Horizontal, symbol Device:D_ALT
- J_DC_INT1: footprint Connector_Molex:Molex_KK-254_1x02_P2.54mm_Horizontal -> Connector_Molex:Molex_KK-254_AE-6410-02A_1x02_P2.54mm_Vertical
Connections:
- wire segments 54 -> 38
Other:
- note added: "Utiliser un L293D (D = Diodes incluses)"
