File: Action_Level/PCB/Action_Card_Sensors-Part.sch (KiCad schematic (older format))
At the start: 4 parts

Commit message: End of the schematic
Parts:
- removed J_FC_R: Conn_01x02, symbol Connector_Generic:Conn_01x02
- added J_FC_LB1, J_FC_RB1, J_FC_RT1: Conn_01x02, Connector_Molex:Molex_KK-254_1x02_P2.54mm_Horizontal, symbol Connector_Generic:Conn_01x03
- added U1: txb0108, Package_SO:TSSOP-20_4.4x6.5mm_P0.65mm, symbol stm32f042k6tx:txb0108
- J_FC_LT1: renamed from J_FC_L; footprint (none) -> Connector_Molex:Molex_KK-254_1x02_P2.54mm_Horizontal; symbol Connector_Generic:Conn_01x02 -> Connector_Generic:Conn_01x03
- J_SENSOR_AR1: renamed from J_TR_AR; footprint (none) -> Connector_Molex:Molex_KK-254_1x04_P2.54mm_Horizontal; symbol Connector_Generic:Conn_01x04 -> Connector_Generic:Conn_01x03
- J_SENSOR_AV1: renamed from J_TR_AV; footprint (none) -> Connector_Molex:Molex_KK-254_1x04_P2.54mm_Horizontal; symbol Connector_Generic:Conn_01x04 -> Connector_Generic:Conn_01x03
Connections:
- net labels added: +5V, FC_LB, FC_LT, FC_RB, FC_RT, GND, SENSOR_AR, SENSOR_AV
- net labels removed: +3V3, FC_L, FC_R
Other:
- note added: "Capteurs fin de courses (2 en haut + 2 en bas)"
- note added: "Capteurs présence palet (1 pour le palet avant et 1 pour le palet arrière)"

Commit message: First big step in route
Parts:
- J_FC_LB1, J_FC_LT1, J_FC_RB1, J_FC_RT1: footprint Connector_Molex:Molex_KK-254_1x02_P2.54mm_Horizontal -> Connector_Molex:Molex_KK-254_AE-6410-03A_1x03_P2.54mm_Vertical
- J_SENSOR_AR1, J_SENSOR_AV1: footprint Connector_Molex:Molex_KK-254_1x04_P2.54mm_Horizontal -> Connector_Molex:Molex_KK-254_AE-6410-03A_1x03_P2.54mm_Vertical
Changed lines of the file:
@@
 F 0 "J_FC_LT1" H 4200 2300 50  0000 C CNN
 F 1 "Conn_01x02" H 4225 2400 50  0000 C CNN
-F 2 "Connector_Molex:Molex_KK-254_1x02_P2.54mm_Horizontal" H 3925 2375 50  0001 C CNN
+F 2 "Connector_Molex:Molex_KK-254_AE-6410-03A_1x03_P2.54mm_Vertical" H 3925 2375 50  0001 C CNN
 F 3 "~" H 3925 2375 50  0001 C CNN
 	1    3925 2375
@@
 F 0 "J_SENSOR_AV1" H 4225 4525 50  0000 C CNN
 F 1 "Conn_01x04" H 4225 4600 50  0000 C CNN
-F 2 "Connector_Molex:Molex_KK-254_1x04_P2.54mm_Horizontal" H 3900 4600 50  0001 C CNN
+F 2 "Connector_Molex:Molex_KK-254_AE-6410-03A_1x03_P2.54mm_Vertical" H 3900 4600 50  0001 C CNN
 F 3 "~" H 3900 4600 50  0001 C CNN
 	1    3900 4600
@@
 F 0 "J_SENSOR_AR1" H 4225 5075 50  0000 C CNN
 F 1 "Conn_01x04" H 4225 5150 50  0000 C CNN
-F 2 "Connector_Molex:Molex_KK-254_1x04_P2.54mm_Horizontal" H 3900 5150 50  0001 C CNN
+F 2 "Connector_Molex:Molex_KK-254_AE-6410-03A_1x03_P2.54mm_Vertical" H 3900 5150 50  0001 C CNN
 F 3 "~" H 3900 5150 50  0001 C CNN
 	1    3900 5150
@@
 F 0 "J_FC_RT1" H 4200 3025 50  0000 C CNN
 F 1 "Conn_01x02" H 4225 3125 50  0000 C CNN
-F 2 "Connector_Molex:Molex_KK-254_1x02_P2.54mm_Horizontal" H 3925 3100 50  0001 C CNN
+F 2 "Connector_Molex:Molex_KK-254_AE-6410-03A_1x03_P2.54mm_Vertical" H 3925 3100 50  0001 C CNN
 F 3 "~" H 3925 3100 50  0001 C CNN
 	1    3925 3100
@@
 F 0 "J_FC_LB1" H 6150 2300 50  0000 C CNN
 F 1 "Conn_01x02" H 6175 2400 50  0000 C CNN
-F 2 "Connector_Molex:Molex_KK-254_1x02_P2.54mm_Horizontal" H 5875 2375 50  0001 C CNN
+F 2 "Connector_Molex:Molex_KK-254_AE-6410-03A_1x03_P2.54mm_Vertical" H 5875 2375 50  0001 C CNN
 F 3 "~" H 5875 2375 50  0001 C CNN
 	1    5875 2375
@@
 F 0 "J_FC_RB1" H 6150 3025 50  0000 C CNN
 F 1 "Conn_01x02" H 6175 3125 50  0000 C CNN
-F 2 "Connector_Molex:Molex_KK-254_1x02_P2.54mm_Horizontal" H 5875 3100 50  0001 C CNN
+F 2 "Connector_Molex:Molex_KK-254_AE-6410-03A_1x03_P2.54mm_Vertical" H 5875 3100 50  0001 C CNN
 F 3 "~" H 5875 3100 50  0001 C CNN
 	1    5875 3100
