File: Action_Level/PCB/Action_Card_Power-Part.sch (KiCad schematic (older format))
At the start: 35 parts

Commit message: End of the schematic
Parts:
- added J_FAN1: Conn_01x02, Connector_Molex:Molex_KK-254_1x02_P2.54mm_Horizontal, symbol Connector_Generic:Conn_01x02
- C10, C7, C9: renamed from C?; footprint (none) -> Capacitor_THT:CP_Radial_D8.0mm_P3.50mm
- C11, C12, C8: renamed from C?; footprint (none) -> Capacitor_SMD:C_1206_3216Metric_Pad1.42x1.75mm_HandSolder
- Cin_1: footprint (none) -> Capacitor_SMD:C_1206_3216Metric_Pad1.42x1.75mm_HandSolder
- Cin_2: renamed from Cin_?; footprint (none) -> Capacitor_SMD:C_1206_3216Metric_Pad1.42x1.75mm_HandSolder
- Cin_3, Cin_4: renamed from Cin_?; footprint (none) -> Capacitor_THT:CP_Radial_D8.0mm_P3.50mm
- D10, D11, D12: renamed from D?; footprint (none) -> Diode_THT:D_DO-35_SOD27_P10.16mm_Horizontal
- D13, D14, D15, D16, D17: renamed from D?; footprint (none) -> LED_SMD:LED_1206_3216Metric_Pad1.42x1.75mm_HandSolder
- F1, F2, F3: renamed from F?; footprint (none) -> Fuse:Fuse_1206_3216Metric_Pad1.42x1.75mm_HandSolder
- R10, R11, R3, R4, R5, R6, R7, R8, R9: renamed from R?; footprint (none) -> Resistor_SMD:R_1206_3216Metric_Pad1.42x1.75mm_HandSolder
- U5, U6, U7: renamed from U?; footprint (none) -> B plug:B plug 5mm
- U8, U9: renamed from U?; footprint Package_TO_SOT_SMD:SOT-223 -> Package_TO_SOT_SMD:SOT-223-3_TabPin2
Connections:
- wire segments 66 -> 70
Other:
- note added: "Connecteur ventilateur\n"

Commit message: First big step in route
Parts:
- D10, D11, D12: footprint Diode_THT:D_DO-35_SOD27_P10.16mm_Horizontal -> Diode_SMD:D_SMA_Handsoldering
- J_FAN1: footprint Connector_Molex:Molex_KK-254_1x02_P2.54mm_Horizontal -> Connector_Molex:Molex_KK-254_AE-6410-02A_1x02_P2.54mm_Vertical
Changed lines of the file:
@@
 F 0 "D10" V 4375 2325 50  0000 L CNN
 F 1 "D_10A" H 4275 2150 50  0000 L CNN
-F 2 "Diode_THT:D_DO-35_SOD27_P10.16mm_Horizontal" H 4375 2250 50  0001 C CNN
+F 2 "Diode_SMD:D_SMA_Handsoldering" H 4375 2250 50  0001 C CNN
 F 3 "~" H 4375 2250 50  0001 C CNN
 	1    4375 2250
@@
 F 0 "D11" V 4975 4775 50  0000 L CNN
 F 1 "D_10A" H 4875 4600 50  0000 L CNN
-F 2 "Diode_THT:D_DO-35_SOD27_P10.16mm_Horizontal" H 4975 4700 50  0001 C CNN
+F 2 "Diode_SMD:D_SMA_Handsoldering" H 4975 4700 50  0001 C CNN
 F 3 "~" H 4975 4700 50  0001 C CNN
 	1    4975 4700
@@
 F 0 "D12" V 4975 5875 50  0000 L CNN
 F 1 "D_10A" H 4875 5700 50  0000 L CNN
-F 2 "Diode_THT:D_DO-35_SOD27_P10.16mm_Horizontal" H 4975 5800 50  0001 C CNN
+F 2 "Diode_SMD:D_SMA_Handsoldering" H 4975 5800 50  0001 C CNN
 F 3 "~" H 4975 5800 50  0001 C CNN
 	1    4975 5800
@@
 F 0 "J_FAN1" H 8055 4942 50  0000 L CNN
 F 1 "Conn_01x02" H 8055 4851 50  0000 L CNN
-F 2 "Connector_Molex:Molex_KK-254_1x02_P2.54mm_Horizontal" H 7975 4950 50  0001 C CNN
+F 2 "Connector_Molex:Molex_KK-254_AE-6410-02A_1x02_P2.54mm_Vertical" H 7975 4950 50  0001 C CNN
 F 3 "~" H 7975 4950 50  0001 C CNN
 	1    7975 4950

Commit message: Debug of route part + 3dshapes
Parts:
- U5, U6, U7: footprint B plug:B plug 5mm -> B plug:Bplug-5mm
Changed lines of the file:
@@
 F 0 "U5" H 3300 2300 60  0000 C CNN
 F 1 "B_Plug_5mm" H 3275 2000 60  0000 C CNN
-F 2 "B plug:B plug 5mm" H 3400 2150 60  0001 C CNN
+F 2 "B plug:Bplug-5mm" H 3400 2150 60  0001 C CNN
 F 3 "" H 3400 2150 60  0000 C CNN
 	1    3400 2150
@@
 F 0 "U6" H 3900 4750 60  0000 C CNN
 F 1 "B_Plug_5mm" H 3450 4600 60  0000 C CNN
-F 2 "B plug:B plug 5mm" H 4000 4600 60  0001 C CNN
+F 2 "B plug:Bplug-5mm" H 4000 4600 60  0001 C CNN
 F 3 "" H 4000 4600 60  0000 C CNN
 	1    4000 4600
@@
 F 0 "U7" H 3900 5850 60  0000 C CNN
 F 1 "B_Plug_5mm" H 3450 5700 60  0000 C CNN
-F 2 "B plug:B plug 5mm" H 4000 5700 60  0001 C CNN
+F 2 "B plug:Bplug-5mm" H 4000 5700 60  0001 C CNN
 F 3 "" H 4000 5700 60  0000 C CNN
 	1    4000 5700
